File: schematic_NEMA23/schematic_NEMA23.kicad_sch (KiCad schematic)
At the start: 123 parts, among them IC1 TB67S249FTG,EL, IC2 STM32L433CCU6, IC3 TJA1441AT_0Z, J1 CAN (1=CANH,2=CANL,3=GND), J10 Conn_01x05, J11 POWER 12-24V / >=10A (1=VIN,2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, J2 CAN (1=CANH,2=CANL,3=GND), J3 MOTOR A+/A-/B-/B+, J4 MOTOR A+/A-/B-/B+, J5 SWD / SWO, J6 5077CR-16SMC2-BK-TR, J7 POWER 12-24V / >=10A (1=VIN,2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, J8 POWER 12-24V / >=10A (1=VIN,2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, J9 SENS I2C (3V3/GND/SCL/SDA), SW2 KHS42E, U2 AP63205WU, U3 USBLC6-2P6, U4 TPS2116DRLR, U5 NCP360, U6 AP2112K-3.3TRG1

Commit message: NEMA17/23 回路図に電線注記を追加し R32 を DNP に変更
- 両回路図の J3/J4 付近に、モーター出力の電線選定に関する注記を追加
  - AWG22 は 3A 定格で余裕がないため、3A 付近で運転する場合は J4 を使い、電線は AWG18 以上にする
  - J3 と J4 は同じ出力を並列に出すため、同時に 2 台のモーターは接続しない
- NEMA23 の TH1 の Value を Thermistor_NTC から NCP18XH103F03RB に変更
- 両回路図の R32 を dnp no から dnp yes に変更
- NEMA23 の kicad_pro で used_designators の並びを整理（指定の内容は変更なし）
- NEMA23 の ERC 結果（schematic_NEMA23-erc.json）を追加

Co-Authored-By: Claude Sonnet 5.5 <noreply@anthropic.com>
Parts:
- R32: now not fitted
- TH1: value Thermistor_NTC -> NCP18XH103F03RB
Other:
- note added: "AWG22 で 3A 定格のため、3A 運転では余裕がない。 3A 付近で運転する場合は J4（JST VH B4P-VH、AWG16 で 10A 定格）を使い、 電線は AWG18 以上にする。J3 と J4 は同じ出力を並列に出すコネクタなので、 同時に 2 台のモーターはつながない |"
Changed lines of the file:
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@@
 		)
 	)
+	(text "AWG22 で 3A 定格のため、3A 運転では余裕がない。\n3A 付近で運転する場合は J4（JST VH B4P-VH、AWG16 で 10A 定格）を使い、\n電線は AWG18 以上にする。J3 と J4 は同じ出力を並列に出すコネクタなので、\n同時に 2 台のモーターはつながない |"
+		(exclude_from_sim no)
+		(at 250.698 526.034 0)
+		(effects
+			(font
+				(size 1.27 1.27)
+			)
+		)
+	)
 	(text "USB only: MCU on, motor VM off.\nUSB current before enumeration <=100mA total.\nVM = ADC/4095 * VDDA * 19; wait >=10ms after power changes.\n4.5A is driver absolute peak maximum; initial VREF limit ~1.97A/phase.\nRoute high-current PGND via NT1 only; keep BUCK_SW away from ADC.\nAP2112 dissipation and motor/Q1 cooling require thermal validation."
 		(exclude_from_sim no)
@@
 			)
 		)
-		(property "Value" "Thermistor_NTC"
+		(property "Value" "NCP18XH103F03RB"
 			(at 128.27 192.0874 0)
 			(show_name no)
@@
 		(on_board yes)
 		(in_pos_files yes)
-		(dnp no)
+		(dnp yes)
 		(property "Reference" "R32"
 			(at 305.562 471.424 0)
